Commit message: fixed to deal with upside-down botasensor

File: poli2_description/urdf/j2s7s300_robotiq_botasensor.xacro (robot description, xacro)
@@ -164,5 +164,5 @@
 	  <parent link="${prefix}_link_7"/>
 	  <child link="ft_sensor0_wrench"/>
-	  <origin xyz="0 0 -0.055" rpy="0 ${J_PI} ${J_PI/2}" />
+	  <origin xyz="0 0 -0.055" rpy="0 -${J_PI} -${J_PI/2}" />
 	</joint>
 	<link name="ft_sensor0_wrench" />
@@ -170,5 +170,5 @@
 	  <parent link="${prefix}_link_7"/>
 	  <child link="ft_sensor0_imu" />
-	  <origin xyz="0 0 -0.055" rpy="0 ${J_PI} ${J_PI/2}" />
+	  <origin xyz="0 0 -0.055" rpy="0 -${J_PI} -${J_PI/2}" />
 	</joint>
 	<link name ="ft_sensor0_imu" />
