Commit message: changed name of botasensor, changed tf tree, added launch option to start bota sensor from machine1

File: poli2_description/robots/poli2_freight.urdf.xacro (robot description, xacro)
@@ -39,5 +39,5 @@
     <xacro:include filename="$(find poli2_description)/urdf/poli_components/neck_mount.urdf.xacro"/>
     <!-- using the f/t sensor we will need this arm urdf-->
-    <xacro:include filename="$(find poli2_description)/urdf/j2s7s300_robotiq_bota.xacro" />
+    <xacro:include filename="$(find poli2_description)/urdf/j2s7s300_robotiq_botasensor.xacro" />
     <xacro:property name="M_PI" value="3.14159"/>
     <xacro:property name="HALF_PI" value="1.57079"/>

File: poli2_description/urdf/j2s7s300_robotiq.xacro (robot description, xacro)
@@ -163,8 +163,8 @@
 	<joint name="bota_ftsensor_joint" type="fixed">
 	  <parent link="${prefix}_link_7"/>
-	  <child link="bota_ftsensor_wrench" />
+	  <child link="ftsensor0_wrench" />
 	  <origin xyz="0 0 -0.055" rpy="0 ${J_PI} ${J_PI/2}" />
 	</joint>
-	<link name="bota_ftsensor_wrench" />
+	<link name="ftsensor0_wrench" />
         <link name="${prefix}_ee_link"/>
 	<joint name="${prefix}_ee_gripper" type="fixed">

File: poli2_description/urdf/j2s7s300_robotiq_botasensor.xacro (robot description, xacro)
@@ -163,14 +163,14 @@
 	<joint name="bota_ftsensor_joint" type="fixed">
 	  <parent link="${prefix}_link_7"/>
-	  <child link="bota_ftsensor_wrench"/>
+	  <child link="ft_sensor0_wrench"/>
 	  <origin xyz="0 0 -0.055" rpy="0 ${J_PI} ${J_PI/2}" />
 	</joint>
-	<link name="bota_ftsensor_wrench" />
+	<link name="ft_sensor0_wrench" />
 	<joint name="bota_ftsensor_joint2" type="fixed">
 	  <parent link="${prefix}_link_7"/>
-	  <child link="bota_ftsensor_imu" />
+	  <child link="ft_sensor0_imu" />
 	  <origin xyz="0 0 -0.055" rpy="0 ${J_PI} ${J_PI/2}" />
 	</joint>
-	<link name ="bota_ftsensor_imu" />
+	<link name ="ft_sensor0_imu" />
         <link name="${prefix}_ee_link"/>
 	<joint name="${prefix}_ee_gripper" type="fixed">
